File: poe-only-top-smt/pizero-poe.sch (KiCad schematic (older format))
At the start: 69 parts, among them IC1 ENC28J60-I/ML, J1 RJ45-LED, P1 Raspberry_Pi_+_Conn, P2 WS2812 Cn., P3 WS2812 Cn., Q1 SI3440DV, Q3 BSS138, T1 PULSE_H1197, T2 TRANSFO, T3 VOLTAGE_REF, U1 LTC4267, U2 PAS291, U3 LM1117IMPX-ADJ, Y1 25Mhz

Commit message: use rpi interface from ihartwig/raspberrypi-debugger and footprints from kicad 4+
Parts:
- removed C17: CP, w_smd_cap:c_elec_8x6.5, symbol CP
- removed C19: 0.1uf, w_smd_cap:c_0402, symbol C
- removed C20: 1uf, w_smd_cap:c_0402, symbol C
- removed D6: LED, w_smd_leds:Led_0603, symbol LED
- removed D7: ZENER, w_smd_diode:sod123, symbol ZENER
- removed P1: Raspberry_Pi_+_Conn, symbol Raspberry_Pi_+_Conn
- removed P2: WS2812 Cn., w_pin_strip:pin_strip_3, symbol CONN_01X03
- removed P3: WS2812 Cn., w_pin_strip:pin_strip_3-90, symbol CONN_01X03
- removed Q3: BSS138, w_smd_trans:sot23, symbol BSS138
- removed R13: 390, w_smd_resistors:r_0402, symbol R
- removed R15: 240, w_smd_resistors:r_0402, symbol R
- removed R18: 360, w_smd_resistors:r_0402, symbol R
- removed R23, R24: 14k, w_smd_resistors:r_0402, symbol R
- removed R25: 100, w_smd_resistors:r_0402, symbol R
- removed U3: LM1117IMPX-ADJ, w_smd_trans:sot223, symbol LM1117IMPX-ADJ
- added C17: dnp-100n, Capacitors_SMD:C_0603, symbol C_Small
- added C19, C20: 1uF, Capacitors_SMD:C_0603, symbol C_Small
- added D6, D7: LED Green, LEDs:LED_0603, symbol Led_Small
- added H1, H2, H3, H4: hole-metalized-no4, pizero-poe-special:hole-m3, symbol hole-metalized-no4
- added P1: dnp-CONN_01X02, Pin_Headers:Pin_Header_Straight_1x02, symbol CONN_01X02
- added P2: dnp-REF-182665-01, pizero-poe-special:Pin_Header_Straight_TH-SMT-NoPaste_2x20, symbol CONN_02X20
- added Q2: DMMT3906_Dual_PNP, TO_SOT_Packages_SMD:SOT-23-6, symbol DMMT3906_Dual_PNP
- added Q3: Q_PMOS_GSD, TO_SOT_Packages_SMD:SOT-23, symbol Q_PMOS_GSD
- added R13: 1k, Resistors_SMD:R_0603, symbol R_Small
- added R15: 10k, Resistors_SMD:R_0603, symbol R_Small
- added R18: dnp-1k, Resistors_SMD:R_0603, symbol R_Small
- added R19: 47k, Resistors_SMD:R_0603, symbol R_Small
- added R20, R23: dnp-3.9k, Resistors_SMD:R_0603, symbol R_Small
- added R24: 220, Resistors_SMD:R_0603, symbol R_Small
- added U3: dnp-AT24CS32-SSHM, Housings_SSOP:TSSOP-8_4.4x3mm_Pitch0.65mm, symbol AT24CS32-SSHM
- added U4: AP7365_SOT-23-5, TO_SOT_Packages_SMD:SOT-23-5, symbol AP7365_SOT-23-5
- C1, C14, C18, C2, C21, C3, C6, C7, C8, C9: footprint w_smd_cap:c_0402 -> Capacitors_SMD:C_0603
- C10, C11, C13, C15, C16: footprint w_smd_cap:c_0603 -> Capacitors_SMD:C_0603
- C12: footprint w_smd_cap:c_elec_4x4.5 -> Capacitors_SMD:c_elec_4x4.5
- C22: footprint w_smd_cap:c_0805 -> Capacitors_SMD:C_1206
- C4: footprint w_smd_cap:c_tant_B -> Capacitors_SMD:c_elec_4x4.5
- C5: footprint w_smd_cap:c_tant_D -> Capacitors_SMD:C_1206
- D1, D2: footprint w_smd_diode:MBS -> pizero-poe-special:MBS
- D3: footprint w_smd_diode:do214ac -> pizero-poe-special:sod523
- D4: footprint w_smd_diode:sod523 -> pizero-poe-special:sod523
- D5: footprint w_smd_diode:do214ab -> pizero-poe-special:sod523
- IC1: footprint w_smd_qfn:qfn-28 -> Housings_DFN_QFN:QFN-28-1EP_6x6mm_Pitch0.65mm; Mouser Part No. 579-ENC28J60-I/ML -> (none)
- L1: footprint w_smd_inductors:inductor_smd_1008 -> Resistors_SMD:R_1206
- L2: footprint w_smd_inductors:inductor_smd_0402 -> Resistors_SMD:R_0603
- Q1: footprint w_smd_trans:tsot-6 -> TO_SOT_Packages_SMD:SOT-23-6
- R1, R10, R11, R12, R14, R16, R17, R2, R21, R22, R26, R3, R4, R5, R7, R8, R9: footprint w_smd_resistors:r_0402 -> Resistors_SMD:R_0603
- R6: footprint w_smd_resistors:r_1206 -> Resistors_SMD:R_1206
- T3: footprint w_smd_trans:sot23 -> TO_SOT_Packages_SMD:SOT-23
- U1: footprint w_smd_dil:ssop-16 -> Housings_SSOP:QSOP-16_3.9x4.9mm_Pitch0.635mm
Connections:
- net labels added: +3V3, GPIO0_ID_SD, GPIO10_MOSI, GPIO11_SCLK, GPIO12, GPIO13, GPIO14_TXD0, GPIO15_RXD0, GPIO16_CE2#, GPIO17, GPIO18, GPIO19, GPIO1_ID_SC, GPIO1_SDA1, GPIO20_MOSI, GPIO21_SCLK, GPIO22, GPIO23, GPIO24, GPIO25, GPIO26, GPIO27, GPIO3_SCL1, GPIO4, GPIO5, GPIO6, GPIO7_CE1#, GPIO8_CE0#, GPIO9_MISO, GPIO_25, RPI_3V3_1, RPI_3V3_2, RPI_VBUS
- net labels removed: ENC_CS, ENC_INT, ENC_SCK, ENC_SI, ENC_SO, ENC_WOL, WS2812_DO
- wire segments 276 -> 307
- no-connect marks 2 -> 6
Other:
- note added: "16-bit addressed I2C EEPROM, 32Kb+\nStores RPi HAT configuration."
- note added: "Extra Linear Reg. for 3.3V\n\nPower ethernet phy whether we\nhave PoE or not. Phy requires more\npower than allowed from RPi 3.3V."
- note added: "Ideal Diode for RPi 5V Source\n\nQ1: Low Rds PFET like DMP3099L.\n3A, 99mΩ @ 4.5V Vgs.\nQ2: Matched PNP pair. Current mirror\ncomparator pulls Q1 gate low (on)\nwhen USB_VBUS_RVP > USB_VBUS."
- note added: "Raspberry Pi Power"
- note added: "TH Female Bottom or SMT Female Top Header\nSMT: Toby Electronics REF-182665-01/REF-182665-03\nTH: Digikey 1528-1385-ND\nPin #s Match RPi."
- note removed: "Linear Regulator"
- note removed: "WS2812 Driver"

Commit message: floorplan, named nets, design rules set
Parts:
- removed C4: 220uf, Capacitors_SMD:c_elec_4x4.5, symbol CP
- removed P1: dnp-CONN_01X02, Pin_Headers:Pin_Header_Straight_1x02, symbol CONN_01X02
- added C23, C25, C4: 2.2uF 100V, Capacitors_SMD:C_1206, symbol C
- added C24: 0.1uF 100V, Capacitors_SMD:C_0603, symbol C
- added W1, W2, W3: TEST_1P, Measurement_Points:Measurement_Point_Round-SMD-Pad_Small, symbol TEST_1P
- C1: value 0.1uf -> 0.1uf 100V
- C11: footprint Capacitors_SMD:C_0603 -> Capacitors_SMD:C_1206
- C12: value CP -> 470uF
- C15, C16: value 0.1uf -> 0.1uF
- C22: value 1uf -> 2.2uF 100V
- C5: value 6.8uf -> 2.2uF 100V
- C6: value C -> DNP
- D3: value ZENER -> SMAJ58A; footprint pizero-poe-special:sod523 -> Diodes_SMD:DO-214BA
- D5: value D_Schottky -> SBM1040; footprint pizero-poe-special:sod523 -> Diodes_SMD:DO-214BA
- R5: value R -> DNP
Connections:
- net labels added: LEDA_A, LEDA_K, LEDB_A, LEDB_K, PHY_OSC1, PHY_OSC2, POE_FB_A, POE_FB_DIV, POE_FB_K, POE_PVCC, POE_RUN, POE_SW_D, POE_SW_SENSE, POE_VPORTN, POE_VPORTP, POE_VPORTP_L, POW_SW_S, TPIN_T+, TPIN_T-, TPOUT_T+, TPOUT_T-, ~POE_PWRGD
- net labels removed: LEDA_CATH, LEDB_CATH, PVCC, RUN
- wire segments 307 -> 321
Other:
- moved on the sheet: C13, C22, C5, C6, R5

Commit message: complete routing for poe and ethernet
* isolate to ~500Vac with .75-.8mm gaps between high and low voltage copper
* remove extra 2x13 compatibility holes from pizero_poe_special:Pin_Header_Straight_TH-SMT-NoPaste_2x20, Pin_Header_Straight_TH-SMT_2x20 footprints
* add insert attribute to pizero_poe_special:Crystal_Grounded_3.2x2.5, MBS, Pin_Header_Straight_TH-SMT_2x20, sod123, sod323, sod523 footprints.
* change rpi hat eeprom power from RPI_3V3_2 to +3V3
* calculate trace geometry for ethenet impedance control
Parts:
- removed C6: DNP, Capacitors_SMD:C_0603, symbol C
- removed R5: DNP, Resistors_SMD:R_0603, symbol R
- removed W3: TEST_1P, Measurement_Points:Measurement_Point_Round-SMD-Pad_Small, symbol TEST_1P
- added D8: LED Green, LEDs:LED_0603, symbol Led_Small
- added R5: 23k, Resistors_SMD:R_0603, symbol R_Small
Connections:
- net labels removed: GPIO_25
- wire segments 321 -> 322

Commit message: add datasheets, change eth magnetics, clean up silkscreen
Parts:
- removed T1: PULSE_H1197, project_foot:H2019, symbol PULSE_H1197
- added T1: H2019FNL, pizero-poe-special:Transformer_Pulse_H2019FNL, symbol H2019FNL
- D3: Description (none) -> TVS DIODE 58VWM 93.6VC SMA; Digikey Part No (none) -> SMAJ58ALFCT-ND; Mfg (none) -> Littelfuse; Mfg Part No (none) -> SMAJ58A; Type (none) -> SMT
- J1: Description (none) -> Jack Modular Connector 8p8c (RJ45, Ethernet) 90° Angle (Rig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; Digikey Part No (none) -> RJHSE-5081-ND; Mfg (none) -> Amphenol; Mfg Part No (none) -> RJHSE-5081; Type (none) -> TH
- R21, R22: Type (none) -> SMT
Connections:
- wire segments 322 -> 326
Other:
- note added: "Open drain LEDs set default\nto full-duplex on reset."
- moved on the sheet: C21, R17, R26

Commit message: add part info to schematic for BOM. TODO: UPDATE LAYOUT
Parts:
- C1: Description (none) -> 0.10µF 100V Ceramic Capacitor X7R 0603; Digikey Part No (none) -> 1276-6807-1-ND; Mfg (none) -> Samsung; Mfg Part No (none) -> CL10B104KC8NNNC; Mouser Part No. 710-885012105001 -> (none); Type (none) -> SMT
- C10, C15, C16, C18, C21, C7, C8, C9: Mouser Part No. 710-885012105001 -> (none); Type (none) -> SMT
- C11: Mouser Part No. 81-ZRB18AR61C106ME1L -> (none); Type (none) -> SMT
- C12: footprint Capacitors_SMD:c_elec_4x4.5 -> Capacitors_SMD:c_elec_8x10; Description (none) -> 470µF 10V Aluminum Capacitors Radial, Can - SMD; Digikey Part No (none) -> 493-2169-1-ND; Mfg (none) -> Nichicon; Mfg Part No (none) -> UWT1A471MNL1GS; Mouser Part No. 667-EEE-1AA330WR -> (none); Type (none) -> SMT
- C13: value 2nf -> 2.2nF 250Vac; Description (none) -> 2200pF 250V Ceramic Capacitor C0G, NP0 0603; Digikey Part No (none) -> 445-15244-1-ND; Mfg (none) -> TDK Corporation; Mfg Part No (none) -> C1608C0G2E222J080AA; Mouser Part No. 81-GRM1885C1H202JA1D -> (none); Type (none) -> SMT
- C14: Mouser Part No. 81-GRM155R71H682KA8D -> (none); Type (none) -> SMT
- C17: value dnp-100n -> nostuff-0.1u; Type (none) -> nostuff
- C19, C20, R13, R15, R19, R24, R5, R9: Type (none) -> SMT
- C2, C3: Mouser Part No. 81-GRM1555C1H160JA1D -> (none); Type (none) -> SMT
- C22: Description (none) -> 2.2µF 100V Ceramic Capacitor X7R 1206; Digikey Part No (none) -> 490-7209-1-ND; Mfg (none) -> Murata Electronics; Mfg Part No (none) -> GRM31CR72A225KA73L; Mouser Part No. 810-C2012X7S2A105K -> (none); Type (none) -> SMT
- C23, C25, C4, C5: Description (none) -> 2.2µF 100V Ceramic Capacitor X7R 1206; Digikey Part No (none) -> 490-7209-1-ND; Mfg (none) -> Murata Electronics; Mfg Part No (none) -> GRM31CR72A225KA73L; Mouser Part No. 74-293D685X9050D2TE3 -> (none); Type (none) -> SMT
- C24: Description (none) -> 0.10µF 100V Ceramic Capacitor X7R 0603; Digikey Part No (none) -> 1276-6807-1-ND; Mfg (none) -> Samsung; Mfg Part No (none) -> CL10B104KC8NNNC; Mouser Part No. 810-C2012X7S2A105K -> (none); Type (none) -> SMT
- D1, D2: Description (none) -> Bridge Rectifier Single Phase 100V 800mA Surface Mount 4-Mi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; Digikey Part No (none) -> HD01DICT-ND; Mfg (none) -> Diodes Inc; Mfg Part No (none) -> HD01-T; Mouser Part No. 621-HD01-T -> (none); Type (none) -> SMT
- D4: Description (none) -> Diode Standard 100V 250mA (DC) Surface Mount SOD-523; Digikey Part No (none) -> 568-1603-1-ND; Mfg (none) -> NXP Semiconductors; Mfg Part No (none) -> BAS516,115; Type (none) -> SMT
- D5: Description (none) -> Diode Schottky 150V 3A Surface Mount PMDS; Digikey Part No (none) -> RB058L150TE25CT-ND; Mfg (none) -> Rohm Semiconductor; Mfg Part No (none) -> RB058L150TE25; Mouser Part No. 621-B360A-F -> (none); Type (none) -> SMT
- D6, D7, D8: Description (none) -> LED GREEN CLEAR 0603 SMD; Digikey Part No (none) -> 160-1183-1-ND; Mfg (none) -> Lite-On; Mfg Part No (none) -> LTST-C190GKT; Type (none) -> SMT
- H1, H2, H3, H4, P2, W1, W2: Type (none) -> nostuff
- IC1: Digikey Part No (none) -> ENC28J60-I/ML-ND; Mfg (none) -> Microchip Technology; Mfg Part No (none) -> ENC28J60-I/ML; Type (none) -> SMT
- J1: Mouser Part No. 710-615008137421 -> (none)
- L1: Description (none) -> 2.2µH Unshielded Multilayer Inductor 1.3A 188 mOhm Max 1008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; Digikey Part No (none) -> 490-10966-1-ND; Mfg (none) -> Murata Electronics; Mfg Part No (none) -> LQM2HPN2R2MEHL; Type (none) -> SMT
- L2: Mouser Part No. 81-BLM15AG102SN1D -> (none); Type (none) -> SMT
- Q1: Description (none) -> MOSFET N-CH 150V 1.2A 6-TSOP; Digikey Part No (none) -> SI3440DV-T1-E3CT-ND; Mfg (none) -> Vishay Siliconix; Mfg Part No (none) -> SI3440DV-T1-E3; Type (none) -> SMT
- Q2: Description (none) -> TRANS 2PNP 40V 0.2A SOT26; Digikey Part No (none) -> DMMT3906-7-FDICT-ND; Mfg (none) -> Diodes Inc; Mfg Part No (none) -> DMMT3906-7-F; Type (none) -> SMT
- Q3: Description (none) -> MOSFET P-CH 30V SOT23; Digikey Part No (none) -> DMP3099L-7DICT-ND; Mfg (none) -> Diodes Inc; Mfg Part No (none) -> DMP3099L-7; Type (none) -> SMT
- R1: value DNP -> nostuff; Type (none) -> nostuff
- R10, R11, R2, R4: Mouser Part No. 754-RR0510P-103D -> (none); Type (none) -> SMT
- R12: Mouser Part No. 754-RR0510P-332D -> (none); Type (none) -> SMT
- R14, R16, R17, R26: Mouser Part No. 660-RK73H1ETQTP49R9F -> (none); Type (none) -> SMT
- R18: value dnp-1k -> nostuff-1k; Type (none) -> nostuff
- R20, R23: value dnp-3.9k -> nostuff-3.9k; Type (none) -> nostuff
- R21, R22: Mouser Part No. 667-ERJ-2RKF5490X -> (none)
- R3: Mouser Part No. 754-RR0510P-102D -> (none); Type (none) -> SMT
- R6: Description (none) -> RES SMD 0.05 OHM 1% 1W 1206; Digikey Part No (none) -> CSNL1206FT50L0CT-ND; Mfg (none) -> Stackpole Electronics; Mfg Part No (none) -> CSNL1206FT50L0; Type (none) -> SMT
- R7: Mouser Part No. 754-RR0510P-682D -> (none); Type (none) -> SMT
- R8: Mouser Part No. 667-ERJ-2RKF2321X -> (none); Type (none) -> SMT
- T1: Alt Mfg (none) -> Pulse Electronics; Alt Mfg Part No (none) -> H2019FNL; Description (none) -> TRANS WE-LAN 10/100 POE SMD; Digikey Part No (none) -> 732-7063-1-ND; Mfg (none) -> Wurth Electronics Inc; Mfg Part No (none) -> 749013011A; Type (none) -> SMT
- T2: Description (none) -> TRANS FLYBACK POE 127UH SMD; Digikey Part No (none) -> 732-2433-1-ND; Mfg (none) -> Wurth Electronics Inc; Mfg Part No (none) -> 7491199501; Type (none) -> SMT
- T3: Description (none) -> Shunt Voltage Reference IC 16V ±0.5% 20mA SOT-23-3 (TO-236); Digikey Part No (none) -> TLV431BSN1T1GOSCT-ND; Mfg (none) -> ON Semiconductor; Mfg Part No (none) -> TLV431BSN1T1G; Type (none) -> SMT
- U1: Description (none) -> Power Over Ethernet Controller 1 Channel 802.3af (PoE) 16-S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; Digikey Part No (none) -> LTC4267CGN-3#PBF-ND; Digikey Part No. LTC4267CGN-3#PBF-ND -> (none); Mfg (none) -> Linear Technology; Mfg Part No (none) -> LTC4267CGN#PBF; Type (none) -> SMT
- U2: value PAS291 -> PS2911-1-K-AX; Description (none) -> Optoisolator Transistor Output 2500Vrms 1 Channel 4-Mini-Fl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; Digikey Part No (none) -> PS2911-1-K-AX-ND; Mfg (none) -> CEL; Mfg Part No (none) -> PS2911-1-K-AX; Type (none) -> SMT
- U3: value dnp-AT24CS32-SSHM -> nostuff-AT24CS32-SSHM; Type (none) -> nostuff
- U4: Description (none) -> Linear Voltage Regulator IC Positive Fixed 1 Output 3.3V 60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; Digikey Part No (none) -> AP7365-33WG-7DICT-ND; Mfg (none) -> Diodes Inc; Mfg Part No (none) -> AP7365-33WG-7; Type (none) -> SMT
- Y1: Digikey Part No (none) -> CTX1175CT-ND; Mfg (none) -> CTS Frequency Controls; Mfg Part No (none) -> 445I23D25M00000; Type (none) -> SMT

Commit message: fix layout for larger cap, isolation, solder mask
* larger footprint for 470uF cap and adjust power and phy to fit
* fix 3d model of rpi header for 20 pins
* add soldermask expansion
* allow soldermask tenting on ethernet phy ep
* add gerbers
Parts:
- C13: footprint Capacitors_SMD:C_0603 -> Capacitors_SMD:C_1812; Description 2200pF 250V Ceramic Capacitor C0G, NP0 0603 -> 2200pF 250VAC Ceramic Capacitor X7R 1812; Digikey Part No 445-15244-1-ND -> 732-10345-1-ND; Mfg TDK Corporation -> Wurth Electronics; Mfg Part No C1608C0G2E222J080AA -> 885362211015
- L2: Description (none) -> FERRITE BEAD 1 KOHM 0603 1LN; Digikey Part No (none) -> 587-1867-1-ND; Mfg (none) -> Taiyo Yuden; Mfg Part No (none) -> BK1608HS102-T
- T2: Alt Mfg (none) -> Wurth Electronics Inc; Alt Mfg Part No (none) -> 7491199501; Description TRANS FLYBACK POE 127UH SMD -> XFRMR 5V 13.5W 127UH POE EP13; Digikey Part No 732-2433-1-ND -> 553-1983-1-ND; Mfg Wurth Electronics Inc -> Pulse Electronics; Mfg Part No 7491199501 -> PA1137NLT
Changed lines of the file:
@@
 F 0 "C13" H 8875 10400 50  0000 L CNN
 F 1 "2.2nF 250Vac" H 8875 10200 50  0000 L CNN
-F 2 "Capacitors_SMD:C_0603" H 8888 10150 50  0001 C CNN
+F 2 "Capacitors_SMD:C_1812" H 8888 10150 50  0001 C CNN
 F 3 "" H 8850 10300 50  0000 C CNN
 F 4 "SMT" H 8850 10300 60  0001 C CNN "Type"
-F 5 "TDK Corporation" H 8850 10300 60  0001 C CNN "Mfg"
-F 6 "C1608C0G2E222J080AA" H 8850 10300 60  0001 C CNN "Mfg Part No"
-F 7 "445-15244-1-ND" H 8850 10300 60  0001 C CNN "Digikey Part No"
-F 8 "2200pF 250V Ceramic Capacitor C0G, NP0 0603" H 8850 10300 60  0001 C CNN "Description"
+F 5 "Wurth Electronics" H 8850 10300 60  0001 C CNN "Mfg"
+F 6 "885362211015" H 8850 10300 60  0001 C CNN "Mfg Part No"
+F 7 "732-10345-1-ND" H 8850 10300 60  0001 C CNN "Digikey Part No"
+F 8 "2200pF 250VAC Ceramic Capacitor X7R 1812" H 8850 10300 60  0001 C CNN "Description"
 	1    8850 10300
 	0    1    1    0
@@
 F 4 "710-7491199501" H 8850 7750 60  0001 C CNN "Mouser Part No."
 F 5 "SMT" H 8850 7750 60  0001 C CNN "Type"
-F 6 "Wurth Electronics Inc" H 8850 7750 60  0001 C CNN "Mfg"
-F 7 "7491199501" H 8850 7750 60  0001 C CNN "Mfg Part No"
-F 8 "732-2433-1-ND" H 8850 7750 60  0001 C CNN "Digikey Part No"
-F 9 "TRANS FLYBACK POE 127UH SMD" H 8850 7750 60  0001 C CNN "Description"
+F 6 "Pulse Electronics" H 8850 7750 60  0001 C CNN "Mfg"
+F 7 "PA1137NLT" H 8850 7750 60  0001 C CNN "Mfg Part No"
+F 8 "553-1983-1-ND" H 8850 7750 60  0001 C CNN "Digikey Part No"
+F 9 "XFRMR 5V 13.5W 127UH POE EP13" H 8850 7750 60  0001 C CNN "Description"
+F 10 "Wurth Electronics Inc" H 8850 7750 60  0001 C CNN "Alt Mfg"
+F 11 "7491199501" H 8850 7750 60  0001 C CNN "Alt Mfg Part No"
 	1    8850 7750
 	1    0    0    -1
@@
 F 3 "" H 5300 1300 50  0000 C CNN
 F 4 "SMT" V 5300 1300 60  0001 C CNN "Type"
+F 5 "Taiyo Yuden" V 5300 1300 60  0001 C CNN "Mfg"
+F 6 "BK1608HS102-T" V 5300 1300 60  0001 C CNN "Mfg Part No"
+F 7 "587-1867-1-ND" V 5300 1300 60  0001 C CNN "Digikey Part No"
+F 8 "FERRITE BEAD 1 KOHM 0603 1LN" V 5300 1300 60  0001 C CNN "Description"
 	1    5300 1300
 	-1   0    0    1

Commit message: update readme, bom, gerbers
Parts:
- C13: Alt Mfg (none) -> Wurth Electronics; Alt Mfg Part No (none) -> 885362211015; Digikey Part No 732-10345-1-ND -> 490-3492-1-ND; Mfg Wurth Electronics -> Murata; Mfg Part No 885362211015 -> GA343QR7GD222KW01L
- R5: value 23k -> 22k
Changed lines of the file:
@@
 F 3 "" H 8850 10300 50  0000 C CNN
 F 4 "SMT" H 8850 10300 60  0001 C CNN "Type"
-F 5 "Wurth Electronics" H 8850 10300 60  0001 C CNN "Mfg"
-F 6 "885362211015" H 8850 10300 60  0001 C CNN "Mfg Part No"
-F 7 "732-10345-1-ND" H 8850 10300 60  0001 C CNN "Digikey Part No"
+F 5 "Murata" H 8850 10300 60  0001 C CNN "Mfg"
+F 6 "GA343QR7GD222KW01L" H 8850 10300 60  0001 C CNN "Mfg Part No"
+F 7 "490-3492-1-ND" H 8850 10300 60  0001 C CNN "Digikey Part No"
 F 8 "2200pF 250VAC Ceramic Capacitor X7R 1812" H 8850 10300 60  0001 C CNN "Description"
+F 9 "Wurth Electronics" H 8850 10300 60  0001 C CNN "Alt Mfg"
+F 10 "885362211015" H 8850 10300 60  0001 C CNN "Alt Mfg Part No"
 	1    8850 10300
 	0    1    1    0
@@
 P 5250 8000
 F 0 "R5" H 5280 8020 50  0000 L CNN
-F 1 "23k" H 5280 7960 50  0000 L CNN
+F 1 "22k" H 5280 7960 50  0000 L CNN
 F 2 "Resistors_SMD:R_0603" H 5250 8000 50  0001 C CNN
 F 3 "" H 5250 8000 50  0000 C CNN
